File: CANcapable.kicad_sch (KiCad schematic)
At the start: 29 parts, among them J1 USB_C_Receptacle_USB2.0_14P, J10 Conn_01x05, J2 Screw_Terminal_01x03, U1 STM32G431C8Tx, U2 SN65HVD230, U4 L78L33_SOT89

Commit message: added missing symbols
Parts:
- added C19, C20, C21, C22, C23, C24: 100nF, Capacitor_SMD:C_0603_1608Metric_Pad1.08x0.95mm_HandSolder, symbol Device:C_Small
- added C25: 4.7uF, Capacitor_SMD:C_0603_1608Metric_Pad1.08x0.95mm_HandSolder, symbol Device:C_Small
- added R4, R6: 5K1, Resistor_SMD:R_0603_1608Metric_Pad0.98x0.95mm_HandSolder, symbol Device:R_Small
Connections:
- net +3.3V: now also C19.1, C20.1, C21.1, C22.1, C23.1, C24.1, C25.1
- net +5V: now also J1.A4 (VBUS), J1.A9 (VBUS), J1.B4 (VBUS), J1.B9 (VBUS)
- net GND: now also J1.A1 (GND), J1.A12 (GND), J1.B1 (GND), J1.B12 (GND), J1.S1 (SHIELD), U1.19 (VSSA), U1.23 (VSS), U1.35 (VSS), U1.47 (VSS), C19.2, C20.2, C21.2, C22.2, C23.2, C24.2, C25.2, R4.2, R6.2
- net CC1: now reaches J1.A5 (CC1)
- net CC1: now also R6.1
- net USB_DP: now reaches J1.A6 (D+)
- net USB_DP: now also J1.B6 (D+)
- net USB_DN: now reaches J1.A7 (D-)
- net USB_DN: now also J1.B7 (D-)
- net CC2: now reaches J1.B5 (CC2)
- net CC2: now also R4.1
Other:
- note added: "100nF for evey VDD and 4.7uF at common point"
- note added: "Decoupling"
- moved on the sheet: J2, U1

Commit message: begin layout
Parts:
- added C8: 100nF, Capacitor_SMD:C_0603_1608Metric_Pad1.08x0.95mm_HandSolder, symbol Device:C_Small
- added J1: USB header, Connector_PinHeader_2.54mm:PinHeader_1x04_P2.54mm_Vertical, symbol Connector_Generic:Conn_01x04
- added JP3: SolderJumper_2_Open, Connector_PinHeader_2.54mm:PinHeader_1x02_P2.54mm_Vertical, symbol Jumper:SolderJumper_2_Open
- added R7: 10k, Resistor_SMD:R_0603_1608Metric_Pad0.98x0.95mm_HandSolder, symbol Device:R_Small
- J2: renamed from J1; footprint (none) -> Connector_USB:USB_C_Receptacle_HRO_TYPE-C-31-M-12
- R1: value 100k -> 10k
- renumbered C14 to C1, C22 to C10, C23 to C11, C24 to C12, C25 to C13, C15 to C2, C16 to C3, C1 to C4, C19 to C5, C3 to C6, C20 to C7, C21 to C9, D4 to D1, D3 to D2, D2 to D3, H5 to H1, H6 to H2, H7 to H3, H8 to H4, J10 to J3, J2 to J4, R5 to R10, R4 to R2, R6 to R3, R15 to R4, R14 to R5, R13 to R6, R2 to R8, R3 to R9, U4 to U1, U1 to U2, U2 to U3
Connections:
- net FDCAN1_RX is gone; now on net BOOT0: U3.4 (R)
- net +3.3V: now also C4.1, C6.1, U2.1 (VBAT), U2.20 (VREF+), U2.21 (VDDA), U2.24 (VDD), U2.36 (VDD), U2.48 (VDD), R7.1
- net +3V3D: no longer C4.1, C6.1
- net +5V: now also J1.4 (Pin_4)
- net BOOT0: now also U2.45 (PB8)
- net CAN_1_H: now also J4.2 (Pin_2)
- net CAN_1_L: now also J4.3 (Pin_3), JP3.1 (A); no longer R10.2
- net FDCAN1_TX: now also U2.46 (PB9)
- net GND: now also J4.1 (Pin_1), C8.2, J1.1 (Pin_1)
- net NRST: now also U2.7 (PG10), C8.1, R7.2
- net STAT_LED: now also U2.39 (PA15)
- net SWCLK: now also U2.38 (PA14)
- net SWDIO: now also U2.37 (PA13)
- net USB_DN: now also U2.34 (PA12), J1.3 (Pin_3)
- net USB_DP: now also U2.33 (PA11), J1.2 (Pin_2)
- new net: JP3.2 (B), R10.2
Other:
- moved on the sheet: J4, R10, R2, R3
